File: bc-module-epaper.brd (EAGLE design)
At the start: 88 x 55 mm, 47 parts, among them J1 SFV24R-4STE1HLF, Q1 PMV30UN2, U1 TCA9534PW, U2 SN74AHC1G32DBV, U3 TS12A44514PW, U4 TPS22917DBV

Commit message: Add files via upload
Parts:
- moved C4 0.10 mm to (44.0, 18.6), turned to 180 degrees
- turned C2 to 180 degrees
- turned R3 to 180 degrees
Routing:
- net GND: track 0.00 -> 45.9 mm, vias 0 -> 13
- net RESE: track 49.3 -> 50.4 mm
- net VDD: track 60.1 -> 60.8 mm
- added copper zone on layer 1, net GND
Other:
- board text added: "by VPetras"
